Commit message: WIP: figuring out how to spawn in half_sitting

File: talos_harmonic/models/talos_description/talos.urdf (robot description, URDF)
Before this commit: robot talos, 82 links, 81 joints
Links:
- link arm_left_1_link: geometry collision mesh filename=package://talos_description/meshes/arm/arm_1_collision.STL scale=1 1 1; visual mesh filename=package://talos_description/meshes/arm/arm_1.STL scale=1 1 1
- link arm_left_2_link: geometry collision mesh filename=package://talos_description/meshes/arm/arm_2_collision.STL scale=1 1 1; visual mesh filename=package://talos_description/meshes/arm/arm_2.STL scale=1 1 1
- link arm_left_3_link: geometry collision mesh filename=package://talos_description/meshes/arm/arm_3_collision.STL scale=1 1 1; visual mesh filename=package://talos_description/meshes/arm/arm_3.STL scale=1 1 1
- link arm_left_4_link: geometry collision mesh filename=package://talos_description/meshes/arm/arm_4_collision.STL scale=1 1 1; visual mesh filename=package://talos_description/meshes/arm/arm_4.STL scale=1 1 1
- link arm_left_5_link: geometry collision mesh filename=package://talos_description/meshes/arm/arm_5_collision.STL scale=1 1 1; visual mesh filename=package://talos_description/meshes/arm/arm_5.STL scale=1 1 1
- link arm_left_6_link: geometry collision mesh filename=package://talos_description/meshes/arm/arm_6_collision.STL scale=1 1 1; visual mesh filename=package://talos_description/meshes/arm/arm_6.STL scale=1 1 1
- link arm_left_7_link: geometry collision mesh filename=package://talos_description/meshes/arm/arm_7_collision.STL scale=1 1 1; visual mesh filename=package://talos_description/meshes/arm/arm_7.STL scale=1 1 1
- link arm_right_1_link: geometry collision mesh filename=package://talos_description/meshes/arm/arm_1_collision.STL scale=1 -1 1; visual mesh filename=package://talos_description/meshes/arm/arm_1.STL scale=1 -1 1
- link arm_right_2_link: geometry collision mesh filename=package://talos_description/meshes/arm/arm_2_collision.STL scale=1 -1 1; visual mesh filename=package://talos_description/meshes/arm/arm_2.STL scale=1 -1 1
- link arm_right_3_link: geometry collision mesh filename=package://talos_description/meshes/arm/arm_3_collision.STL scale=1 -1 1; visual mesh filename=package://talos_description/meshes/arm/arm_3.STL scale=1 -1 1
- link arm_right_4_link: geometry collision mesh filename=package://talos_description/meshes/arm/arm_4_collision.STL scale=1 -1 1; visual mesh filename=package://talos_description/meshes/arm/arm_4.STL scale=1 -1 1
- link arm_right_5_link: geometry collision mesh filename=package://talos_description/meshes/arm/arm_5_collision.STL scale=1 -1 1; visual mesh filename=package://talos_description/meshes/arm/arm_5.STL scale=1 -1 1
- link arm_right_6_link: geometry collision mesh filename=package://talos_description/meshes/arm/arm_6_collision.STL scale=1 -1 1; visual mesh filename=package://talos_description/meshes/arm/arm_6.STL scale=1 -1 1
- link arm_right_7_link: geometry collision mesh filename=package://talos_description/meshes/arm/arm_7_collision.STL scale=1 -1 1; visual mesh filename=package://talos_description/meshes/arm/arm_7.STL scale=1 -1 1
- link base_link: geometry collision mesh filename=package://talos_description/meshes/torso/base_link_collisio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 scale=1 1 1; visual mesh filename=package://talos_description/meshes/torso/base_link.STL scale=1 1 1
- link gripper_left_base_link: geometry collision mesh filename=package://talos_description/meshes/gripper/base_link_collis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 scale=1 1 1; visual mesh filename=package://talos_description/meshes/gripper/base_link.STL scale=1 1 1
- link gripper_left_fingertip_1_link: geometry collision mesh filename=package://talos_description/meshes/gripper/fingertip_collis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 scale=1 1 1; visual mesh filename=package://talos_description/meshes/gripper/fingertip.STL scale=1 1 1
- link gripper_left_fingertip_2_link: geometry collision mesh filename=package://talos_description/meshes/gripper/fingertip_collis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 scale=1 1 1; visual mesh filename=package://talos_description/meshes/gripper/fingertip.STL scale=1 1 1
- link gripper_left_fingertip_3_link: geometry collision mesh filename=package://talos_description/meshes/gripper/fingertip_collis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 scale=1 1 1; visual mesh filename=package://talos_description/meshes/gripper/fingertip.STL scale=1 1 1
- link gripper_left_inner_double_link: geometry collision mesh filename=package://talos_description/meshes/gripper/inner_double_col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 scale=1 1 1; visual mesh filename=package://talos_description/meshes/gripper/inner_double.STL scale=1 1 1
- link gripper_left_inner_single_link: geometry collision mesh filename=package://talos_description/meshes/gripper/inner_single_col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 scale=1 1 1; visual mesh filename=package://talos_description/meshes/gripper/inner_single.STL scale=1 1 1
- link gripper_left_motor_double_link: geometry collision mesh filename=package://talos_description/meshes/gripper/gripper_motor_do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 scale=1 1 1; visual mesh filename=package://talos_description/meshes/gripper/gripper_motor_do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 scale=1 1 1
- link gripper_left_motor_single_link: geometry collision mesh filename=package://talos_description/meshes/gripper/gripper_motor_si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 scale=1 1 1; visual mesh filename=package://talos_description/meshes/gripper/gripper_motor_si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 scale=1 1 1
- link gripper_right_base_link: geometry collision mesh filename=package://talos_description/meshes/gripper/base_link_collis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 scale=1 1 1; visual mesh filename=package://talos_description/meshes/gripper/base_link.STL scale=1 1 1
- link gripper_right_fingertip_1_link: geometry collision mesh filename=package://talos_description/meshes/gripper/fingertip_collis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 scale=1 1 1; visual mesh filename=package://talos_description/meshes/gripper/fingertip.STL scale=1 1 1
- link gripper_right_fingertip_2_link: geometry collision mesh filename=package://talos_description/meshes/gripper/fingertip_collis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 scale=1 1 1; visual mesh filename=package://talos_description/meshes/gripper/fingertip.STL scale=1 1 1
- link gripper_right_fingertip_3_link: geometry collision mesh filename=package://talos_description/meshes/gripper/fingertip_collis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 scale=1 1 1; visual mesh filename=package://talos_description/meshes/gripper/fingertip.STL scale=1 1 1
- link gripper_right_inner_double_link: geometry collision mesh filename=package://talos_description/meshes/gripper/inner_double_col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 scale=1 1 1; visual mesh filename=package://talos_description/meshes/gripper/inner_double.STL scale=1 1 1
- link gripper_right_inner_single_link: geometry collision mesh filename=package://talos_description/meshes/gripper/inner_single_col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 scale=1 1 1; visual mesh filename=package://talos_description/meshes/gripper/inner_single.STL scale=1 1 1
- link gripper_right_motor_double_link: geometry collision mesh filename=package://talos_description/meshes/gripper/gripper_motor_do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 scale=1 1 1; visual mesh filename=package://talos_description/meshes/gripper/gripper_motor_do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 scale=1 1 1
- link gripper_right_motor_single_link: geometry collision mesh filename=package://talos_description/meshes/gripper/gripper_motor_si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 scale=1 1 1; visual mesh filename=package://talos_description/meshes/gripper/gripper_motor_si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 scale=1 1 1
- link head_1_link: geometry collision mesh filename=package://talos_description/meshes/head/head_1_collision.stl scale=1 1 1; visual mesh filename=package://talos_description/meshes/head/head_1.stl scale=1 1 1
- link head_2_link: geometry collision mesh filename=package://talos_description/meshes/head/head_2_default_coll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 scale=1 1 1; visual mesh filename=package://talos_description/meshes/head/head_2_default.stl scale=1 1 1
- link leg_left_1_link: geometry collision mesh filename=package://talos_description/meshes/v2/hip_z_collision.stl scale=1 1 1; visual mesh filename=package://talos_description/meshes/v2/hip_z_lo_res.stl scale=1 1 1
- link leg_left_2_link: geometry collision mesh filename=package://talos_description/meshes/v2/hip_x_collision.stl scale=1 1 1; visual mesh filename=package://talos_description/meshes/v2/hip_x_lo_res.stl scale=1 1 1
- link leg_left_3_link: geometry collision mesh filename=package://talos_description/meshes/v2/hip_y_collision.stl scale=1 1 1; visual mesh filename=package://talos_description/meshes/v2/hip_y_lo_res.stl scale=1 1 1
- link leg_left_4_link: geometry collision mesh filename=package://talos_description/meshes/v2/knee_collision.stl scale=1 1 1; visual mesh filename=package://talos_description/meshes/v2/knee_lo_res.stl scale=1 1 1
- link leg_left_5_link: geometry collision mesh filename=package://talos_description/meshes/v2/ankle_Y_collision.stl scale=1 1 1; visual mesh filename=package://talos_description/meshes/v2/ankle_Y_lo_res.stl scale=1 1 1
- link leg_left_6_link: geometry collision mesh filename=package://talos_description/meshes/v2/ankle_X_collision.stl scale=1.15 1.05 1; visual mesh filename=package://talos_description/meshes/v2/ankle_X_lo_res.stl scale=1 1 1
- link leg_right_1_link: geometry collision mesh filename=package://talos_description/meshes/v2/hip_z_collision.stl scale=1 -1 1; visual mesh filename=package://talos_description/meshes/v2/hip_z_lo_res.stl scale=1 -1 1
- link leg_right_2_link: geometry collision mesh filename=package://talos_description/meshes/v2/hip_x_collision.stl scale=1 -1 1; visual mesh filename=package://talos_description/meshes/v2/hip_x_lo_res.stl scale=1 -1 1
- link leg_right_3_link: geometry collision mesh filename=package://talos_description/meshes/v2/hip_y_collision.stl scale=1 -1 1; visual mesh filename=package://talos_description/meshes/v2/hip_y_lo_res.stl scale=1 -1 1
- link leg_right_4_link: geometry collision mesh filename=package://talos_description/meshes/v2/knee_collision.stl scale=1 -1 1; visual mesh filename=package://talos_description/meshes/v2/knee_lo_res.stl scale=1 -1 1
- link leg_right_5_link: geometry collision mesh filename=package://talos_description/meshes/v2/ankle_Y_collision.stl scale=1 -1 1; visual mesh filename=package://talos_description/meshes/v2/ankle_Y_lo_res.stl scale=1 -1 1
- link leg_right_6_link: geometry collision mesh filename=package://talos_description/meshes/v2/ankle_X_collision.stl scale=1.15 -1.05 1; visual mesh filename=package://talos_description/meshes/v2/ankle_X_lo_res.stl scale=1 -1 1
- link torso_1_link: geometry collision mesh filename=package://talos_description/meshes/torso/torso_1.STL scale=1 1 1; visual mesh filename=package://talos_description/meshes/torso/torso_1.STL scale=1 1 1
- link torso_2_link: geometry collision mesh filename=package://talos_description/meshes/torso/torso_2_collision.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 scale=1 1 1; visual mesh filename=package://talos_description/meshes/torso/torso_2.STL scale=1 1 1
